File: PCB/UniAmp.kicad_pcb (KiCad board)
At the start: 2 copper layers, 28.8 x 19.4 mm, 47 parts, among them J1 Conn_01x02_Female, J2 Conn_01x02_Female, J3 Conn_01x05_Female, U1 PIC16F15324, U2 Audio-pcb-rescue_LM49450-Wiib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, U3 LP5907MFX-1.8

Commit message: Some changes
Routing:
- net +3V3: track 60.1 -> 57.5 mm
- net GND: track 53.2 -> 55.5 mm
- net HPS: track 37.6 -> 35.8 mm
Other:
- net class Default: clearance 0.2 -> 0.127; trace_width 0.25 -> 0.127; via_dia 0.8 -> 0.6; via_drill 0.4 -> 0.3
- net class power removed
- rule pad_to_mask_clearance: 0.051 -> 0
- rule solder_mask_min_width: 0.25 -> 0.12
- rule trace_clearance: 0.2 -> 0.127
- rule trace_min: 0.2 -> 0.127
- rule via_min_size: 0.4 -> 0.6
