File: PCB/UniAmp.sch (KiCad schematic (older format))
At the start: 44 parts, among them J1 Conn_01x02_Female, J2 Conn_01x02_Female, J3 Conn_01x05_Female, U1 PIC16F15324, U2 Audio-pcb-rescue_LM49450-Wiib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, U3 LP5907MFX-1.8

Commit message: Some changes
Changed lines of the file:
@@
 EESchema Schematic File Version 4
-LIBS:UniAmp-cache
 EELAYER 30 0
 EELAYER END
@@
 $EndComp
 $Comp
-L power:+3V3 #PWR0113
-U 1 1 5D988CCD
-P 4250 2850
-F 0 "#PWR0113" H 4250 2700 50  0001 C CNN
-F 1 "+3V3" H 4265 3023 50  0000 C CNN
-F 2 "" H 4250 2850 50  0001 C CNN
-F 3 "" H 4250 2850 50  0001 C CNN
-	1    4250 2850
-	-1   0    0    1
-$EndComp
-$Comp
 L Device:C C1
 U 1 1 5D98A4E6
@@
 	1950 2550 2500 2550
 $Comp
-L power:+1V8 #PWR?
+L power:+1V8 #PWR0113
 U 1 1 5DC8DACB
 P 2500 2550
-F 0 "#PWR?" H 2500 2400 50  0001 C CNN
+F 0 "#PWR0113" H 2500 2400 50  0001 C CNN
 F 1 "+1V8" H 2515 2723 50  0000 C CNN
 F 2 "" H 2500 2550 50  0001 C CNN
@@
 Wire Wire Line
 	2500 2550 2900 2550
+$Comp
+L power:+1V8 #PWR0114
+U 1 1 5DC9121F
+P 4250 2850
+F 0 "#PWR0114" H 4250 2700 50  0001 C CNN
+F 1 "+1V8" H 4265 3023 50  0000 C CNN
+F 2 "" H 4250 2850 50  0001 C CNN
+F 3 "" H 4250 2850 50  0001 C CNN
+	1    4250 2850
+	-1   0    0    1
+$EndComp
 $EndSCHEMATC
